File: Hardware/KiCAD/Voltmeter/Voltmeter.kicad_sch (KiCad schematic)
At the start: 29 parts, among them Q1 PMOS, U1 LM397, U2 NME1205DC, U3 ATtiny84A-P, U4 LM397

Commit message: Updated design
Added optocoupler, wiring etc. Updated BoM
Parts:
- added C4, C5: 100nF, symbol Device:C
- added D5: LED, symbol Device:LED
- added Q2: LTV-849, LTV-847_LTO, symbol Optocoupler:LTV-847
- added R17, R18, R19, R20, R21, R22, R23, R24: 220, symbol Device:R
- added U5: MCP3204-CI/P, PDIP14_300MC_MCH, symbol 2024-09-14_22-35-21:MCP3204-CI_P
- C1: value C -> 470nF 600V
- C2: value C -> 100nF
- C3: value C -> 1nF
- R12: value R -> 7.5Meg
- R13: value R -> 4.7Meg
- R14: value R -> 160k
- R15: value R -> 100k
- R16: value R -> 1k
- R2: value R -> 95k
- R9: value R -> 10k
Connections:
- net 5VDCi: now also C4.1, R21.1, R22.1, R23.1, R24.1, U5.13, U5.14; no longer U3.1 (VCC)
- net GND: now also U3.14 (GND), C5.2, R17.2, R18.1, R19.1, R20.1
- net GNDPWR: now also C4.2, Q2.11, Q2.13, Q2.15, U5.12, U5.7; no longer U3.14 (GND)
- net at C1.2, C2.2, C3.2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: no longer R9.2
- net at C2.1, R12.2, U4.3 (+): no longer R9.1
- net freq_detect: now reaches U4.4
- net FREQ_DECT_S: now reaches U3.11 (PA2)
- net DISP_DATA: now reaches U3.12 (PA1)
- net DISP_CLK: now reaches U3.13 (AREF/PA0)
- net at U3.4 (~{RESET}/PB3): now also R9.2
- net LED_CONTROL: now reaches U3.5 (PB2)
- net LED_CONTROL: now also D5.2 (A)
- net SPI_CS: now reaches U3.6 (PA7)
- net SPI_CS: now also Q2.5
- net SPI_MOSI: now reaches U3.7 (PA6)
- net SPI_MOSI: now also Q2.3
- net SPI_MISO: now reaches U3.8 (PA5)
- net SPI_CLK: now reaches U3.9 (PA4)
- net SPI_CLK: now also Q2.1
- new net: Q2.4, R19.2
- new net: D5.1 (K), R17.1
- new net: Q2.2, R20.2
- new net: Q2.6, R18.2
- new net 5VDC: C5.1, R9.1, U3.1 (VCC)
- new net ADC_CH1: U5.1
- new net ADC_CH2: U5.2
- new net ADC_CH3: U5.3
- new net ADC_CH4: U5.4
- new net SPI_CLK_I: Q2.16, R21.2, U5.11
- new net SPI_CS_I: Q2.12, R23.2, U5.8
- new net SPI_MISO_I: U5.10
- new net SPI_MOSI_I: Q2.14, R22.2, U5.9
- no-connect marks 0 -> 8
Other:
- note added: "On the "safe" side of isolation"
- note added: "Will use internal oscillator"
- moved on the sheet: U3

Commit message: Schematic updated
Schematic entry v1 complete
Parts:
- removed R24: 220, symbol Device:R
- added C6: 0.33uF, symbol Device:C
- added C7: 0.1uF, symbol Device:C
- added Q3: LTV-849, LTV-847_LTO, symbol Optocoupler:LTV-847
- added Q4: Q_NPN_CBE, symbol Device:Q_NPN_CBE
- added Q5: Q_NMOS_DGS, symbol Device:Q_NMOS_DGS
- added R25, R26, R29: 220, symbol Device:R
- added R27: 1Meg, symbol Device:R
- added R28: 100k, symbol Device:R
- added R30, R31, R32: 10k, symbol Device:R
- added U6: L7805CV, TO-220_STM, symbol Linear Regulator:L7805CV
- U2: value NME1205DC -> SRS-1205-2; footprint NME_DIP_MUR -> (none)
Connections:
- net 5VDC: now also C7.1, Q3.12, Q3.14, Q3.16, U6.3 (OUTPUT)
- net 5VDCi: now also R21.2, R22.2, R23.2; no longer R21.1, R22.1, R23.1
- net ADC_CH1: now also R3.2, R4.1
- net ADC_CH2: now also Q5.3 (S)
- net ADC_CH3: now also C2.1, R12.2, U4.1 (-)
- net FREQ_DECT_S: now also Q3.15, R30.1
- net GND: now also C6.2, C7.2, R30.2, R31.2, R32.2, U6.2 (GROUND)
- net GNDPWR: now also Q4.3 (E), R25.1, R26.1, R29.1
- net SPI_CLK_I: now also R21.1; no longer R21.2
- net SPI_CS_I: now also R23.1; no longer R23.2
- net SPI_MISO: now also Q3.13, R32.1
- net SPI_MISO_I: now also Q3.3
- net SPI_MOSI_I: now also R22.1; no longer R22.2
- net at D1.1 (K), Q1.3 (S), R.1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: now also R27.1
- net VOLT_RNG_SEL_DC: now reaches U1.4
- net VOLT_RNG_SEL_DC: now also Q3.5, R28.2
- net at R16.1: now also U4.3 (+); no longer U4.1 (-)
- net VOLT_RNG_SEL_DC_S: now reaches U3.10 (PA3)
- net VOLT_RNG_SEL_DC_S: now also Q3.11, R31.1
- net at R5.2, R6.1: now also Q5.1 (D)
- net freq_detect renamed FREQ_DECT
- net FREQ_DECT: now also Q3.1
- new net: Q3.6, R29.2
- new net: Q3.4, R26.2
- new net: Q3.2, R25.2
- new net: Q4.1 (C), Q5.2 (G), R27.2
- new net: Q4.2 (B), R28.1
- new net Vin: C6.1, U6.1 (INPUT)
- no-connect marks 8 -> 12
Other:
- note added: "--> Isolated to Micro zone -->"
- note added: "--> Micro to isolated zone -->"
- note added: "10.8 to 13.2V in"
- note added: "5V to 35V in"
- moved on the sheet: C1, C2, C3, C4, C5, D1, D2, D3, D4, D5, Q1, Q2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

Commit message: Updated parts list and some values, added to digikey list
Updated parts list and some values, added to digikey list
Parts:
- removed R15: 100k, symbol Device:R
- removed U2: SRS-1205-2, symbol 2024-09-10_19-31-40:NME1205DC
- added C8: 6.8uF, symbol Device:C
- added C9: 1uF, symbol Device:C
- added D6: 5.1V, symbol Device:D_Zener
- added D7: 10Vbr, symbol Device:D_Zener
- added U6: RFM-0505S, SIP4_RFM_RCP, symbol Regulator Isolator:RFM-0505S
- C1: renamed from C5; footprint (none) -> Capacitor_THT:C_Axial_L5.1mm_D3.1mm_P15.00mm_Horizontal
- C5: renamed from C3; footprint (none) -> Capacitor_THT:C_Axial_L5.1mm_D3.1mm_P7.50mm_Horizontal
- D4: renamed from D2; value 40Vbr -> 43Vbr
- R1: renamed from R17; footprint (none) -> Resistor_THT:R_Axial_DIN0204_L3.6mm_D1.6mm_P1.90mm_Vertical
- R10: renamed from R2; value 95k -> 95.3k; footprint (none) -> Resistor_THT:R_Axial_DIN0204_L3.6mm_D1.6mm_P1.90mm_Vertical
- R11: renamed from R; footprint (none) -> Resistor_THT:R_Axial_DIN0204_L3.6mm_D1.6mm_P1.90mm_Vertical
- R12: renamed from R28; footprint (none) -> Resistor_THT:R_Axial_DIN0204_L3.6mm_D1.6mm_P1.90mm_Vertical
- R13: footprint (none) -> Resistor_THT:R_Axial_DIN0204_L3.6mm_D1.6mm_P1.90mm_Vertical
- R14: value 160k -> 62k; footprint (none) -> Resistor_THT:R_Axial_DIN0204_L3.6mm_D1.6mm_P1.90mm_Vertical
- R15: renamed from R16; footprint (none) -> Resistor_THT:R_Axial_DIN0204_L3.6mm_D1.6mm_P1.90mm_Vertical
- R17: renamed from R7; value 14M -> 1.4M; footprint (none) -> Resistor_THT:R_Axial_DIN0204_L3.6mm_D1.6mm_P1.90mm_Vertical
- R18: renamed from R8; value 2M -> 200k; footprint (none) -> Resistor_THT:R_Axial_DIN0204_L3.6mm_D1.6mm_P1.90mm_Vertical
- R19: renamed from R11; footprint (none) -> Resistor_THT:R_Axial_DIN0204_L3.6mm_D1.6mm_P1.90mm_Vertical
- R2: renamed from R1; footprint (none) -> Resistor_THT:R_Axial_DIN0204_L3.6mm_D1.6mm_P1.90mm_Vertical
- R20: renamed from R10; footprint (none) -> Resistor_THT:R_Axial_DIN0204_L3.6mm_D1.6mm_P1.90mm_Vertical
- R21: renamed from R20; footprint (none) -> Resistor_THT:R_Axial_DIN0204_L3.6mm_D1.6mm_P1.90mm_Vertical
- R22: renamed from R19; footprint (none) -> Resistor_THT:R_Axial_DIN0204_L3.6mm_D1.6mm_P1.90mm_Vertical
- R23: renamed from R18; footprint (none) -> Resistor_THT:R_Axial_DIN0204_L3.6mm_D1.6mm_P1.90mm_Vertical
- R24: renamed from R25; footprint (none) -> Resistor_THT:R_Axial_DIN0204_L3.6mm_D1.6mm_P1.90mm_Vertical
- R25: renamed from R26; footprint (none) -> Resistor_THT:R_Axial_DIN0204_L3.6mm_D1.6mm_P1.90mm_Vertical
- R26: renamed from R29; footprint (none) -> Resistor_THT:R_Axial_DIN0204_L3.6mm_D1.6mm_P1.90mm_Vertical
- R27: renamed from R30; footprint (none) -> Resistor_THT:R_Axial_DIN0204_L3.6mm_D1.6mm_P1.90mm_Vertical
- R28: renamed from R32; footprint (none) -> Resistor_THT:R_Axial_DIN0204_L3.6mm_D1.6mm_P1.90mm_Vertical
- R29: renamed from R31; footprint (none) -> Resistor_THT:R_Axial_DIN0204_L3.6mm_D1.6mm_P1.90mm_Vertical
- R3: value 20M -> 2M; footprint (none) -> Resistor_THT:R_Axial_DIN0204_L3.6mm_D1.6mm_P1.90mm_Vertical
- R30: renamed from R21; footprint (none) -> Resistor_THT:R_Axial_DIN0204_L3.6mm_D1.6mm_P1.90mm_Vertical
- R31: renamed from R22; footprint (none) -> Resistor_THT:R_Axial_DIN0204_L3.6mm_D1.6mm_P1.90mm_Vertical
- R32: renamed from R23; footprint (none) -> Resistor_THT:R_Axial_DIN0204_L3.6mm_D1.6mm_P1.90mm_Vertical
- R4: value 250k -> 25k; footprint (none) -> Resistor_THT:R_Axial_DIN0204_L3.6mm_D1.6mm_P1.90mm_Vertical
- R5: renamed from R9; footprint (none) -> Resistor_THT:R_Axial_DIN0204_L3.6mm_D1.6mm_P1.90mm_Vertical
- R6: renamed from R5; value 20M -> 2M; footprint (none) -> Resistor_THT:R_Axial_DIN0204_L3.6mm_D1.6mm_P1.90mm_Vertical
- R7: renamed from R6; value 2.85M -> 287k; footprint (none) -> Resistor_THT:R_Axial_DIN0204_L3.6mm_D1.6mm_P1.90mm_Vertical
- R8: renamed from R27; footprint (none) -> Resistor_THT:R_Axial_DIN0204_L3.6mm_D1.6mm_P1.90mm_Vertical
- R9: renamed from R12; footprint (none) -> Resistor_THT:R_Axial_DIN0204_L3.6mm_D1.6mm_P1.90mm_Vertical
- renumbered C1 to C2, C6 to C3, C2 to C4, C7 to C6, C4 to C7, D5 to D1, D1 to D2, D4 to D5, Q4 to Q2, Q5 to Q3, Q2 to Q4, Q3 to Q5, U3 to U1, U5 to U2, U6 to U3, U1 to U5
Connections:
- net 5VDC: now also C8.1, U6.2 (+VIN)
- net 5VDCi: now also C9.1, U6.4 (+VOUT)
- net ADC_CH3: now also R10.1
- net GND: now also C8.2, U6.1 (-VIN)
- net GNDPWR: now also C9.2, D7.2 (A), U6.3 (-VOUT)
- net at C5.1, R13.2, R14.1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: now also D6.1 (K)
- net at C2.2, C4.2, C5.2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: now also D6.2 (A)
- net at Q2.1 (C), Q3.2 (G), R8.2: now also D7.1 (K)
Other:
- note added: "Check this on breadboard"
- moved on the sheet: C4, Q2
